Commit message: Modified URDF and added sdf file for solo
Note:- The sdk still doesnt load solo, there are some gazebo and rviz issues to solve

File: quad_simulator/solo_description/urdf/solo.urdf (robot description, URDF)
Before this commit: robot solo, 17 links, 16 joints
Links:
- link FL_FOOT: geometry collision mesh filename=file:///home/prakhargoel/Desktop/Mitacs/QuadSdk/catkin_ws/s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; visual mesh filename=file:///home/prakhargoel/Desktop/Mitacs/QuadSdk/catkin_ws/s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
- link FL_LOWER_LEG: geometry collision mesh filename=file:///home/prakhargoel/Desktop/Mitacs/QuadSdk/catkin_ws/s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; visual mesh filename=file:///home/prakhargoel/Desktop/Mitacs/QuadSdk/catkin_ws/s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
- link FL_SHOULDER: geometry collision mesh filename=file:///home/prakhargoel/Desktop/Mitacs/QuadSdk/catkin_ws/s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; visual mesh filename=file:///home/prakhargoel/Desktop/Mitacs/QuadSdk/catkin_ws/s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
- link FL_UPPER_LEG: geometry collision mesh filename=file:///home/prakhargoel/Desktop/Mitacs/QuadSdk/catkin_ws/s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; visual mesh filename=file:///home/prakhargoel/Desktop/Mitacs/QuadSdk/catkin_ws/s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
- link FR_FOOT: geometry collision mesh filename=file:///home/prakhargoel/Desktop/Mitacs/QuadSdk/catkin_ws/s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; visual mesh filename=file:///home/prakhargoel/Desktop/Mitacs/QuadSdk/catkin_ws/s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
- link FR_LOWER_LEG: geometry collision mesh filename=file:///home/prakhargoel/Desktop/Mitacs/QuadSdk/catkin_ws/s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; visual mesh filename=file:///home/prakhargoel/Desktop/Mitacs/QuadSdk/catkin_ws/s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
- link FR_SHOULDER: geometry collision mesh filename=file:///home/prakhargoel/Desktop/Mitacs/QuadSdk/catkin_ws/s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; visual mesh filename=file:///home/prakhargoel/Desktop/Mitacs/QuadSdk/catkin_ws/s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
- link FR_UPPER_LEG: geometry collision mesh filename=file:///home/prakhargoel/Desktop/Mitacs/QuadSdk/catkin_ws/s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; visual mesh filename=file:///home/prakhargoel/Desktop/Mitacs/QuadSdk/catkin_ws/s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
- link HL_FOOT: geometry collision mesh filename=file:///home/prakhargoel/Desktop/Mitacs/QuadSdk/catkin_ws/s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; visual mesh filename=file:///home/prakhargoel/Desktop/Mitacs/QuadSdk/catkin_ws/s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
- link HL_LOWER_LEG: geometry collision mesh filename=file:///home/prakhargoel/Desktop/Mitacs/QuadSdk/catkin_ws/s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; visual mesh filename=file:///home/prakhargoel/Desktop/Mitacs/QuadSdk/catkin_ws/s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
- link HL_SHOULDER: geometry collision mesh filename=file:///home/prakhargoel/Desktop/Mitacs/QuadSdk/catkin_ws/s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; visual mesh filename=file:///home/prakhargoel/Desktop/Mitacs/QuadSdk/catkin_ws/s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
- link HL_UPPER_LEG: geometry collision mesh filename=file:///home/prakhargoel/Desktop/Mitacs/QuadSdk/catkin_ws/s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; visual mesh filename=file:///home/prakhargoel/Desktop/Mitacs/QuadSdk/catkin_ws/s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
- link HR_FOOT: geometry collision mesh filename=file:///home/prakhargoel/Desktop/Mitacs/QuadSdk/catkin_ws/s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; visual mesh filename=file:///home/prakhargoel/Desktop/Mitacs/QuadSdk/catkin_ws/s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
- link HR_LOWER_LEG: geometry collision mesh filename=file:///home/prakhargoel/Desktop/Mitacs/QuadSdk/catkin_ws/s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; visual mesh filename=file:///home/prakhargoel/Desktop/Mitacs/QuadSdk/catkin_ws/s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
- link HR_SHOULDER: geometry collision mesh filename=file:///home/prakhargoel/Desktop/Mitacs/QuadSdk/catkin_ws/s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; visual mesh filename=file:///home/prakhargoel/Desktop/Mitacs/QuadSdk/catkin_ws/s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
- link HR_UPPER_LEG: geometry collision mesh filename=file:///home/prakhargoel/Desktop/Mitacs/QuadSdk/catkin_ws/s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; visual mesh filename=file:///home/prakhargoel/Desktop/Mitacs/QuadSdk/catkin_ws/s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
- link base_link: geometry collision mesh filename=file:///home/prakhargoel/Desktop/Mitacs/QuadSdk/catkin_ws/s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; visual mesh filename=file:///home/prakhargoel/Desktop/Mitacs/QuadSdk/catkin_ws/s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

Commit message: Solo now loading in simulation:)
Issue in the zero position when in sit mode, has to be fixed

File: quad_simulator/solo_description/urdf/solo.urdf (robot description, URDF)
Before this commit: robot solo, 17 links, 16 joints
Links:
- removed link FL_FOOT
- removed link FL_LOWER_LEG
- removed link FL_SHOULDER
- removed link FL_UPPER_LEG
- removed link FR_FOOT
- removed link FR_LOWER_LEG
- removed link FR_SHOULDER
- removed link FR_UPPER_LEG
- removed link HL_FOOT
- removed link HL_LOWER_LEG
- removed link HL_SHOULDER
- removed link HL_UPPER_LEG
- removed link HR_FOOT
- removed link HR_LOWER_LEG
- removed link HR_SHOULDER
- removed link HR_UPPER_LEG
- removed link base_link
- added link body, mass 1.16115091; collision mesh filename=file:///home/prakhargoel/Desktop/Mitacs/QuadSdk/catkin_ws/s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; visual mesh filename=file:///home/prakhargoel/Desktop/Mitacs/QuadSdk/catkin_ws/s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
- added link hip0, mass 0.14853845; collision mesh filename=file:///home/prakhargoel/Desktop/Mitacs/QuadSdk/catkin_ws/s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; visual mesh filename=file:///home/prakhargoel/Desktop/Mitacs/QuadSdk/catkin_ws/s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
- added link hip1, mass 0.14853845; collision mesh filename=file:///home/prakhargoel/Desktop/Mitacs/QuadSdk/catkin_ws/s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; visual mesh filename=file:///home/prakhargoel/Desktop/Mitacs/QuadSdk/catkin_ws/s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
- added link hip2, mass 0.14853845; collision mesh filename=file:///home/prakhargoel/Desktop/Mitacs/QuadSdk/catkin_ws/s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; visual mesh filename=file:///home/prakhargoel/Desktop/Mitacs/QuadSdk/catkin_ws/s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
- added link hip3, mass 0.14853845; collision mesh filename=file:///home/prakhargoel/Desktop/Mitacs/QuadSdk/catkin_ws/s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; visual mesh filename=file:///home/prakhargoel/Desktop/Mitacs/QuadSdk/catkin_ws/s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
- added link lower0, mass 0.03070001; collision mesh filename=file:///home/prakhargoel/Desktop/Mitacs/QuadSdk/catkin_ws/s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; visual mesh filename=file:///home/prakhargoel/Desktop/Mitacs/QuadSdk/catkin_ws/s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
- added link lower1, mass 0.03070001; collision mesh filename=file:///home/prakhargoel/Desktop/Mitacs/QuadSdk/catkin_ws/s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; visual mesh filename=file:///home/prakhargoel/Desktop/Mitacs/QuadSdk/catkin_ws/s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
- added link lower2, mass 0.03070001; collision mesh filename=file:///home/prakhargoel/Desktop/Mitacs/QuadSdk/catkin_ws/s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; visual mesh filename=file:///home/prakhargoel/Desktop/Mitacs/QuadSdk/catkin_ws/s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
- added link lower3, mass 0.03070001; collision mesh filename=file:///home/prakhargoel/Desktop/Mitacs/QuadSdk/catkin_ws/s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; visual mesh filename=file:///home/prakhargoel/Desktop/Mitacs/QuadSdk/catkin_ws/s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
- added link toe0, mass 0.00693606; collision mesh filename=file:///home/prakhargoel/Desktop/Mitacs/QuadSdk/catkin_ws/s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; visual mesh filename=file:///home/prakhargoel/Desktop/Mitacs/QuadSdk/catkin_ws/s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
- added link toe1, mass 0.00693606; collision mesh filename=file:///home/prakhargoel/Desktop/Mitacs/QuadSdk/catkin_ws/s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; visual mesh filename=file:///home/prakhargoel/Desktop/Mitacs/QuadSdk/catkin_ws/s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
- added link toe2, mass 0.00693606; collision mesh filename=file:///home/prakhargoel/Desktop/Mitacs/QuadSdk/catkin_ws/s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; visual mesh filename=file:///home/prakhargoel/Desktop/Mitacs/QuadSdk/catkin_ws/s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
- added link toe3, mass 0.00693606; collision mesh filename=file:///home/prakhargoel/Desktop/Mitacs/QuadSdk/catkin_ws/s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; visual mesh filename=file:///home/prakhargoel/Desktop/Mitacs/QuadSdk/catkin_ws/s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
- added link upper0, mass 0.14853845; collision mesh filename=file:///home/prakhargoel/Desktop/Mitacs/QuadSdk/catkin_ws/s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; visual mesh filename=file:///home/prakhargoel/Desktop/Mitacs/QuadSdk/catkin_ws/s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
- added link upper1, mass 0.14853845; collision mesh filename=file:///home/prakhargoel/Desktop/Mitacs/QuadSdk/catkin_ws/s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; visual mesh filename=file:///home/prakhargoel/Desktop/Mitacs/QuadSdk/catkin_ws/s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
- added link upper2, mass 0.14853845; collision mesh filename=file:///home/prakhargoel/Desktop/Mitacs/QuadSdk/catkin_ws/s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; visual mesh filename=file:///home/prakhargoel/Desktop/Mitacs/QuadSdk/catkin_ws/s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
- added link upper3, mass 0.14853845; collision mesh filename=file:///home/prakhargoel/Desktop/Mitacs/QuadSdk/catkin_ws/s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; visual mesh filename=file:///home/prakhargoel/Desktop/Mitacs/QuadSdk/catkin_ws/s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
Joints:
- removed joint FL_ANKLE
- removed joint FL_HAA
- removed joint FL_HFE
- removed joint FL_KFE
- removed joint FR_ANKLE
- removed joint FR_HAA
- removed joint FR_HFE
- removed joint FR_KFE
- removed joint HL_ANKLE
- removed joint HL_HAA
- removed joint HL_HFE
- removed joint HL_KFE
- removed joint HR_ANKLE
- removed joint HR_HAA
- removed joint HR_HFE
- removed joint HR_KFE
- added joint 0: type revolute, parent hip0, child upper0, origin xyz=0 0.014 0 rpy=0 0 0, axis 0 1 0, limit lower=-10 upper=10 effort=1000 velocity=1000
- added joint 1: type revolute, parent upper0, child lower0, origin xyz=0 0.03745 -0.16 rpy=0 0 0, axis 0 1 0, limit lower=-10 upper=10 effort=1000 velocity=1000
- added joint 10: type revolute, parent body, child hip2, origin xyz=0.1946 -0.0875 0 rpy=0 0 0, axis 1 0 0, limit lower=-10 upper=10 effort=1000 velocity=1000
- added joint 11: type revolute, parent body, child hip3, origin xyz=-0.1946 -0.0875 0 rpy=0 0 0, axis 1 0 0, limit lower=-10 upper=10 effort=1000 velocity=1000
- added joint 2: type revolute, parent hip1, child upper1, origin xyz=0 -0.014 0 rpy=0 0 0, axis 0 1 0, limit lower=-10 upper=10 effort=1000 velocity=1000
- added joint 3: type revolute, parent upper1, child lower1, origin xyz=0 -0.03745 -0.16 rpy=0 0 0, axis 0 1 0, limit lower=-10 upper=10 effort=1000 velocity=1000
- added joint 4: type revolute, parent hip2, child upper2, origin xyz=0 -0.014 0 rpy=0 0 0, axis 0 1 0, limit lower=-10 upper=10 effort=1000 velocity=1000
- added joint 5: type revolute, parent upper2, child lower2, origin xyz=0 -0.03745 -0.16 rpy=0 0 0, axis 0 1 0, limit lower=-10 upper=10 effort=1000 velocity=1000
- added joint 6: type revolute, parent hip3, child upper3, origin xyz=0 -0.014 0 rpy=0 0 0, axis 0 1 0, limit lower=-10 upper=10 effort=1000 velocity=1000
- added joint 7: type revolute, parent upper3, child lower3, origin xyz=0 -0.03745 -0.16 rpy=0 0 0, axis 0 1 0, limit lower=-10 upper=10 effort=1000 velocity=1000
- added joint 8: type revolute, parent body, child hip0, origin xyz=0.1946 0.0875 0 rpy=0 0 0, axis 1 0 0, limit lower=-10 upper=10 effort=1000 velocity=1000
- added joint 9: type revolute, parent body, child hip1, origin xyz=0.1946 -0.0875 0 rpy=0 0 0, axis 1 0 0, limit lower=-10 upper=10 effort=1000 velocity=1000
- added joint jtoe0: type fixed, parent lower0, child toe0, origin xyz=0 0.008 -0.16 rpy=0 0 0, limit lower=-10 upper=10 effort=1000 velocity=1000
- added joint jtoe1: type fixed, parent lower1, child toe1, origin xyz=0 -0.008 -0.16 rpy=0 0 0, limit lower=-10 upper=10 effort=1000 velocity=1000
- added joint jtoe2: type fixed, parent lower2, child toe2, origin xyz=0 -0.008 -0.16 rpy=0 0 0, limit lower=-10 upper=10 effort=1000 velocity=1000
- added joint jtoe3: type fixed, parent lower3, child toe3, origin xyz=0 -0.008 -0.16 rpy=0 0 0, limit lower=-10 upper=10 effort=1000 velocity=1000
